Commit message: feat(kuka): refactor KUKA URDF to macro format and implement multi-arm controller configurations in the controller.yaml

File: omnilogix_ws/src/omnilogix_description/kuka_description/urdf/kr16_2.urdf (robot description, URDF)
Before this commit: robot kuka_kr16_2, 9 links, 8 joints
Links:
- removed link base
- removed link base_link
- removed link link_1
- removed link link_2
- removed link link_3
- removed link link_4
- removed link link_5
- removed link link_6
- removed link tool0
Joints:
- removed joint base_link-base
- removed joint joint_a1
- removed joint joint_a2
- removed joint joint_a3
- removed joint joint_a4
- removed joint joint_a5
- removed joint joint_a6
- removed joint joint_a6-tool0
