Commit message: feat(kuka): modularize KUKA arm configuration using XACRO macros and update joint naming conventions for Gazebo integration

File: omnilogix_ws/src/omnilogix_description/kuka_description/urdf/control/kuka.ros2_control.xacro (robot description, xacro)
@@ -1,3 +1,46 @@
 <?xml version="1.0" encoding="UTF-8"?>
-<robot xmlns:xacro ="http://wiki.ros.org/xacro" name="kuka_kr16_2_ros2_control">
+<robot xmlns:xacro ="http://wiki.ros.org/xacro">
+    <xacro:macro name="kuka_kr16_2_ros2_control" params="prefix">
+        <ros2_control name="${prefix}ros2_control" type="system">
+            <hardware>
+                <plugin>gz_ros2_control/GazeboSimSystem</plugin>
+            </hardware>
+            <joint name="${prefix}joint_a1">
+                <command_interface name="position"/>
+                <state_interface name="position"/>
+                <state_interface name="velocity"/>
+                <state_interface name="effort"/>
+            </joint>
+            <joint name="${prefix}joint_a2">
+                <command_interface name="position"/>
+                <state_interface name="position"/>
+                <state_interface name="velocity"/>
+                <state_interface name="effort"/>
+            </joint>
+            <joint name="${prefix}joint_a3">
+                <command_interface name="position"/>
+                <state_interface name="position"/>
+                <state_interface name="velocity"/>
+                <state_interface name="effort"/>
+            </joint>
+            <joint name="${prefix}joint_a4">
+                <command_interface name="position"/>
+                <state_interface name="position"/>
+                <state_interface name="velocity"/>
+                <state_interface name="effort"/>
+            </joint>
+            <joint name="${prefix}joint_a5">
+                <command_interface name="position"/>
+                <state_interface name="position"/>
+                <state_interface name="velocity"/>
+                <state_interface name="effort"/>
+            </joint>
+            <joint name="${prefix}joint_a6">
+                <command_interface name="position"/>
+                <state_interface name="position"/>
+                <state_interface name="velocity"/>
+                <state_interface name="effort"/>
+            </joint>
+        </ros2_control>
+    </xacro:macro>
 </robot>
