Commit message: fix: update joint effort limits in KUKA URDF for improved performance

File: omnilogix_ws/src/omnilogix_description/kuka_description/urdf/description/kr16_2.xacro (robot description, xacro)
@@ -154,5 +154,5 @@
       <child link="${prefix}link_1"/>
       <axis xyz="0 0 -1"/>
-      <limit effort="0" lower="-3.22885911619" upper="3.22885911619" velocity="2.72271363311"/>
+      <limit effort="400" lower="-3.22885911619" upper="3.22885911619" velocity="2.72271363311"/>
     </joint>
     <!-- joint 2 (A2) -->
@@ -162,5 +162,5 @@
       <child link="${prefix}link_2"/>
       <axis xyz="0 1 0"/>
-      <limit effort="0" lower="-2.70526034059" upper="0.610865238198" velocity="2.72271363311"/>
+      <limit effort="400" lower="-2.70526034059" upper="0.610865238198" velocity="2.72271363311"/>
     </joint>
     <!-- joint 3 (A3) -->
@@ -170,5 +170,5 @@
       <child link="${prefix}link_3"/>
       <axis xyz="0 1 0"/>
-      <limit effort="0" lower="-2.26892802759" upper="2.68780704807" velocity="2.72271363311"/>
+      <limit effort="300" lower="-2.26892802759" upper="2.68780704807" velocity="2.72271363311"/>
     </joint>
     <!-- joint 4 (A4) -->
@@ -178,5 +178,5 @@
       <child link="${prefix}link_4"/>
       <axis xyz="-1 0 0"/>
-      <limit effort="0" lower="-6.10865238198" upper="6.10865238198" velocity="5.75958653158"/>
+      <limit effort="100" lower="-6.10865238198" upper="6.10865238198" velocity="5.75958653158"/>
     </joint>
     <!-- joint 5 (A5) -->
@@ -186,5 +186,5 @@
       <child link="${prefix}link_5"/>
       <axis xyz="0 1 0"/>
-      <limit effort="0" lower="-2.26892802759" upper="2.26892802759" velocity="5.75958653158"/>
+      <limit effort="100" lower="-2.26892802759" upper="2.26892802759" velocity="5.75958653158"/>
     </joint>
     <!-- joint 6 (A6) -->
@@ -194,5 +194,5 @@
       <child link="${prefix}link_6"/>
       <axis xyz="-1 0 0"/>
-      <limit effort="0" lower="-6.10865238198" upper="6.10865238198" velocity="10.7337748998"/>
+      <limit effort="50" lower="-6.10865238198" upper="6.10865238198" velocity="10.7337748998"/>
     </joint>
     <!-- tool frame - fixed frame -->
